Commit message: depth and segment filter when creating point cloud

File: tomato_moveit_configs/config/gazebo_ur5e_robot.urdf (robot description, URDF)
Before this commit: robot ur5e_robot, 14 links, 13 joints
Links:
- removed link rob1_cam_link
- added link rob1_cam1_link
- added link rob1_cam2_link
- added link rob1_cam3_link
- added link rob1_cam4_link
- added link rob1_cam_pivot_link
- link rob1_ee_link: geometry collision cylinder length=.16 radius=.08; visual cylinder length=.16 radius=.08
Joints:
- removed joint rob1_ee_cam_joint
- added joint rob1_cam1_joint: type fixed, parent rob1_cam_pivot_link, child rob1_cam1_link, origin xyz=0.0 0.01 0.0 rpy=-1.57079632679 0.0 0.0
- added joint rob1_cam2_joint: type fixed, parent rob1_cam1_link, child rob1_cam2_link, origin xyz=0.01 -0.01 0.0 rpy=0.0 1.57079632679 0.0
- added joint rob1_cam3_joint: type fixed, parent rob1_cam_pivot_link, child rob1_cam3_link, origin xyz=-0.01 0.0 0.0 rpy=0.0 -1.57079632679 0.0
- added joint rob1_cam4_joint: type fixed, parent rob1_cam_pivot_link, child rob1_cam4_link, origin xyz=0.0 -0.01 0.0 rpy=1.57079632679 0.0 0.0
- added joint rob1_ee_cam_pivot_joint: type fixed, parent rob1_ee_link, child rob1_cam_pivot_link, origin xyz=0.0 0.0 0.18 rpy=0.0 0.0 0.0
- joint rob1_wrist_2_joint: origin xyz=0 -0.0997 0 rpy=1.570796327 0 0 -> xyz=0 -0.0997 -2.044881182297852e-11 rpy=1.570796327 0 0
- joint rob1_wrist_3_joint: origin xyz=0 0.0996 0 rpy=1.570796326589793 3.141592653589793 3.141592653589793 -> xyz=0 0.0996 -2.042830148012698e-11 rpy=1.570796326589793 3.141592653589793 3.141592653589793

File: tomato_moveit_configs/urdf/benchbot_sim.urdf.xacro (robot description, xacro)
@@ -36,9 +36,33 @@
         <origin xyz="0.0 0.0 0.00" rpy="0.0 0.0 0.0"/>
     </joint>
-    <link name="rob1_cam_link"/>
-    <joint name="rob1_ee_cam_joint" type="fixed">
+    <link name="rob1_cam_pivot_link"/>
+    <joint name="rob1_ee_cam_pivot_joint" type="fixed">
         <parent link="rob1_ee_link"/>
-        <child link="rob1_cam_link"/>
-        <origin xyz="0.0 0.0 0.01" rpy="0.0 0.0 0.0"/>
+        <child link="rob1_cam_pivot_link"/>
+        <origin xyz="0.0 0.0 0.18" rpy="0.0 0.0 0.0"/>
+    </joint>
+    <link name="rob1_cam1_link"/>
+    <joint name="rob1_cam1_joint" type="fixed">
+        <parent link="rob1_cam_pivot_link"/>
+        <child link="rob1_cam1_link"/>
+        <origin xyz="0.0 0.01 0.0" rpy="-1.57079632679 0.0 0.0"/>
+    </joint>
+    <link name="rob1_cam2_link"/>
+    <joint name="rob1_cam2_joint" type="fixed">
+        <parent link="rob1_cam1_link"/>
+        <child link="rob1_cam2_link"/>
+        <origin xyz="0.01 0.0 -0.01" rpy="0.0 1.57079632679 0.0"/>
+    </joint>
+    <link name="rob1_cam3_link"/>
+    <joint name="rob1_cam3_joint" type="fixed">
+        <parent link="rob1_cam2_link"/>
+        <child link="rob1_cam3_link"/>
+        <origin xyz="0.01 0.0 -0.01" rpy="0.0 1.57079632679 0.0"/>
+    </joint>
+    <link name="rob1_cam4_link"/>
+    <joint name="rob1_cam4_joint" type="fixed">
+        <parent link="rob1_cam3_link"/>
+        <child link="rob1_cam4_link"/>
+        <origin xyz="0.01 0.0 -0.01" rpy="0.0 1.57079632679 0.0"/>
     </joint>
     <xacro:include filename="$(find ur_gazebo)/urdf/ur_macro.xacro"/>
