Commit message: version for conference workshop submission

File: benchbot_multi_eef_moveit_configs/urdf/benchbot_sim.urdf.xacro (robot description, xacro)
@@ -11,5 +11,5 @@
             <origin xyz="0.0 0 0.08" rpy="0.0 0.0 0.0"/>
             <geometry>
-                <cylinder radius=".08" length=".16"/>
+                <cylinder radius=".05" length=".16"/>
             </geometry>
             <material name="White">
@@ -20,5 +20,5 @@
             <origin xyz="0.0 0 0.08" rpy="0.0 0.0 0.0"/>
             <geometry>
-            <cylinder radius=".08" length=".16"/>
+            <cylinder radius=".05" length=".16"/>
             </geometry>
         </collision>
@@ -40,5 +40,5 @@
             <origin xyz="0.0 0 0.08" rpy="0.0 0.0 0.0"/>
             <geometry>
-                <cylinder radius=".08" length=".16"/>
+                <cylinder radius=".05" length=".16"/>
             </geometry>
             <material name="White">
@@ -49,5 +49,5 @@
             <origin xyz="0.0 0 0.08" rpy="0.0 0.0 0.0"/>
             <geometry>
-            <cylinder radius=".08" length=".16"/>
+            <cylinder radius=".05" length=".16"/>
             </geometry>
         </collision>
